File: classic-edition/design/open-amiga-sampler.kicad_sch (KiCad schematic)
At the start: 17 parts, among them J1 Left, J2 Right, J3 DB25_Male, U1 ADC0820CCN, U2 MCP6002-xP^{:3}

Commit message: tweaks, edits, embedded models
Parts:
- removed J1: Left, connectors:Audio pads, symbol Connector:Conn_Coaxial
- removed J2: Right, connectors:Audio pads, symbol Connector:Conn_Coaxial
- added J1: 3.5mm stereo phone, Connector_Audio:Jack_3.5mm_CUI_SJ1-3543, symbol Connector_Audio:AudioJack3
- added unit 1 of U2
- C1: value 10uf^{:2} -> 10uf tantalum^{:2}
- J3: value DB25_Male -> DB25_Pins
- RV1: value R_POT -> 10k expo; footprint connectors:Pot pads -> Potentiometer_Alpha_RD901F-40-00D_Single_Vertical
Connections:
- net AD_IN: now also U2.1; no longer U2.1
- net GND: now also J1.S
- net VCC: now also C3.1, C4.1, J3.14 (P14), U1.12 (VREF(+)), U1.20 (VCC)
- net at R4.1, RV1.1: now also U2.2 (-); no longer U2.2 (-)
- net at C2.1, R5.1, R6.2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: now also U2.3 (+); no longer U2.3 (+)
- net at R2.2: now also J1.R
- net at R1.2: now also J1.T
Other:
- moved on the sheet: C1, R1, R2, R4, RV1
